Commit message: make some updates from NiZiTuFu-Robot

File: src/ranger_mini_v2_gazebo/xacro/ranger_mini_real.xacro (robot description, xacro)
@@ -274,41 +274,41 @@
         </hardware>
         <joint name="fl_wheel">
+            <param name="node_id">-1</param>
+            <command_interface name="velocity">
+            <param name="min">-3.14</param>
+            <param name="max">3.14</param>
+            </command_interface>
+            <state_interface name="velocity"/>
+            <state_interface name="effort"/>
+        </joint>
+        <joint name="fr_wheel">
+            <param name="node_id">6</param>
+            <command_interface name="velocity">
+            <param name="min">-3.14</param>
+            <param name="max">3.14</param>
+            </command_interface>
+            <state_interface name="velocity"/>
+            <state_interface name="effort"/>
+        </joint>
+        <joint name="rl_wheel">
+            <param name="node_id">5</param>
+            <command_interface name="velocity">
+            <param name="min">-3.14</param>
+            <param name="max">3.14</param>
+            </command_interface>
+            <state_interface name="velocity"/>
+            <state_interface name="effort"/>
+        </joint>
+        <joint name="rr_wheel">
+            <param name="node_id">-1</param>
+            <command_interface name="velocity">
+            <param name="min">-3.14</param>
+            <param name="max">3.14</param>
+            </command_interface>
+            <state_interface name="velocity"/>
+            <state_interface name="effort"/>
+        </joint>
+        <joint name="fl_steering_wheel">
             <param name="node_id">1</param>
-            <command_interface name="velocity">
-            <param name="min">-3.14</param>
-            <param name="max">3.14</param>
-            </command_interface>
-            <state_interface name="velocity"/>
-            <state_interface name="effort"/>
-        </joint>
-        <joint name="fr_wheel">
-            <param name="node_id">4</param>
-            <command_interface name="velocity">
-            <param name="min">-3.14</param>
-            <param name="max">3.14</param>
-            </command_interface>
-            <state_interface name="velocity"/>
-            <state_interface name="effort"/>
-        </joint>
-        <joint name="rl_wheel">
-            <param name="node_id">2</param>
-            <command_interface name="velocity">
-            <param name="min">-3.14</param>
-            <param name="max">3.14</param>
-            </command_interface>
-            <state_interface name="velocity"/>
-            <state_interface name="effort"/>
-        </joint>
-        <joint name="rr_wheel">
-            <param name="node_id">3</param>
-            <command_interface name="velocity">
-            <param name="min">-3.14</param>
-            <param name="max">3.14</param>
-            </command_interface>
-            <state_interface name="velocity"/>
-            <state_interface name="effort"/>
-        </joint>
-        <joint name="fl_steering_wheel">
-            <param name="node_id">5</param>
             <command_interface name="position">
             <param name="min">-3.14</param>
@@ -322,5 +322,5 @@
         </joint>
         <joint name="fr_steering_wheel">
-            <param name="node_id">8</param>
+            <param name="node_id">4</param>
             <command_interface name="position">
             <param name="min">-3.14</param>
@@ -334,5 +334,5 @@
         </joint>
         <joint name="rl_steering_wheel">
-            <param name="node_id">6</param>
+            <param name="node_id">2</param>
             <command_interface name="position">
             <param name="min">-3.14</param>
@@ -346,5 +346,5 @@
         </joint>
         <joint name="rr_steering_wheel">
-            <param name="node_id">7</param>
+            <param name="node_id">3</param>
             <command_interface name="position">
             <param name="min">-3.14</param>
